File: Hardware/mmWave-shield-pcb/mmWave-Shield/connectors.kicad_sch (KiCad schematic)
At the start: 4 parts, among them J3 DF40HC_3.0_-40DS-0.4V_51, J4 DF40HC_3.0_-50DS-0.4V_51, J5 DF40C-40DP-0.4V_51, J6 DF40C-50DP-0.4V_51

Commit message: kicad project inital version
Parts:
- J5: footprint Connector_Hirose_DF40:Hirose_DF40HC(3.0)-40DS-0.4V_2x20_P0.4mm -> Connector_Hirose_DF40:Hirose_DF40C-40DS-0.4V_2x20_P0.4mm
- J6: footprint Connector_Hirose_DF40:Hirose_DF40HC(3.0)-50DS-0.4V_2x25_P0.4mm -> Connector_Hirose_DF40:Hirose_DF40C-50DS-0.4V_2x25_P0.4mm
Changed lines of the file:
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@@
 			)
 		)
-		(property "Footprint" "Connector_Hirose_DF40:Hirose_DF40HC(3.0)-50DS-0.4V_2x25_P0.4mm"
+		(property "Footprint" "Connector_Hirose_DF40:Hirose_DF40C-50DS-0.4V_2x25_P0.4mm"
 			(at 223.52 190.17 0)
 			(effects
@@
 			)
 		)
-		(property "Footprint" "Connector_Hirose_DF40:Hirose_DF40HC(3.0)-40DS-0.4V_2x20_P0.4mm"
+		(property "Footprint" "Connector_Hirose_DF40:Hirose_DF40C-40DS-0.4V_2x20_P0.4mm"
 			(at 74.93 196.52 0)
 			(effects

Commit message: Placed Connectors in hopefully right way
Parts:
- J5, J6: now not fitted; now left out of the parts list
Changed lines of the file:
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@@
 		(members "CSI_CLK_N" "CSI_CLK_P" "CSI_D0_N" "CSI_D0_P")
 	)
+	(bus_alias "GAP_GPIOs"
+		(members "GAP_GPIO46" "GAP_GPIO47" "GAP_GPIO50" "GAP_GPIO51" "GAP_GPIO48"
+			"GAP_GPIO49"
+		)
+	)
 	(bus_alias "GPIOs_shared"
 		(members "nRF_P1.00_GAP_GPIO60" "nRF_P1.01_GAP_GPIO61" "nRF_P1.09_GAP_GPIO62"
@@
 		(members "I2C_A_SDA" "I2C_A_SCL" "I2C_B_SDA" "I2C_B_SCL" "I2C_GAP_SEL")
 	)
+	(bus_alias "JTAG_GAP9"
+		(members "VQPS_FUSE_1V8" "RESET_N" "~{TRST}" "TCK" "TCS/CS_RAM_GATE" "TDI"
+			"TDO" "VCC_GAP9"
+		)
+	)
 	(bus_alias "MIC"
 		(members "MIC_DATA" "MIC_CLK" "MIC_THSEL" "MIC_WAKE")
@@
 		)
 	)
+	(bus_alias "QVAR_IMU"
+		(members "QVAR_IMU_1" "QVAR_IMU_2")
+	)
 	(bus_alias "SPI_shared"
 		(members "SPI_A_MOSI" "SPI_A_MISO" "SPI_A_CLK" "SPI_A_CS" "SPI_B_MOSI"
@@
 	(bus_alias "nRF_GPIOs"
 		(members "nRF_P0.04" "nRF_P0.05" "nRF_P0.07" "nRF_P0.25" "nRF_P0.26" "nRF_P0.27"
-			"nRF_P0.31"
+			"nRF_P0.31" "MSP_DR2" "MSP_DR1" "MSP_CS" "nRF_P0.07/AMUX"
+		)
+	)
+	(bus_alias "nRF_QSPI"
+		(members "nRF_QSPI_IO0" "nRF_QSPI_IO1" "nRF_QSPI_IO2" "nRF_QSPI_IO3" "nRF_QSPI_CLK"
+			"nRF_QSPI_CS_CONN" "nRF_QSPI_CS_RAM"
 		)
 	)
@@
 	)
 	(bus_entry
+		(at 57.15 185.42)
+		(size -2.54 2.54)
+		(stroke
+			(width 0)
+			(type default)
+		)
+	)
+	(bus_entry
 		(at 92.71 167.64)
 		(size -2.54 2.54)
@@
 	)
 	(bus_entry
-		(at 57.15 185.42)
-		(size -2.54 2.54)
-		(stroke
-			(width 0)
-			(type default)
-		)
-	)
-	(bus_entry
 		(at 97.79 147.32)
 		(size -2.54 -2.54)
@@
 		)
 	)
-	(bus
-		(pts
-			(xy 57.15 170.18) (xy 57.15 172.72)
-		)
-		(stroke
-			(width 0)
-			(type default)
-		)
-	)
 	(wire
 		(pts
@@
 		)
 	)
-	(bus
-		(pts
-			(xy 57.15 172.72) (xy 57.15 175.26)
-		)
-		(stroke
-			(width 0)
-			(type default)
-		)
-	)
 	(wire
 		(pts
@@
 		)
 	)
-	(bus
-		(pts
-			(xy 57.15 162.56) (xy 57.15 165.1)
-		)
-		(stroke
-			(width 0)
-			(type default)
-		)
-	)
 	(wire
 		(pts
@@
 		)
 	)
-	(wire
+	(bus
 		(pts
-			(xy 175.26 67.31) (xy 194.31 67.31)
+			(xy 57.15 180.34) (xy 57.15 185.42)
 		)
 		(stroke
@@
 		)
 	)
-	(bus
+	(wire
 		(pts
-			(xy 57.15 165.1) (xy 57.15 170.18)
+			(xy 175.26 67.31) (xy 194.31 67.31)
 		)
 		(stroke
@@
 		)
 	)
-	(bus
-		(pts
-			(xy 57.15 175.26) (xy 57.15 177.8)
-		)
-		(stroke
-			(width 0)
-			(type default)
-		)
-	)
 	(wire
 		(pts
@@
 	(wire
 		(pts
+			(xy 53.34 187.96) (xy 54.61 187.96)
+		)
+		(stroke
+			(width 0)
+			(type default)
+		)
+	)
+	(wire
+		(pts
 			(xy 168.91 172.72) (xy 168.91 189.23)
 		)
@@
 		)
 	)
-	(bus
-		(pts
-			(xy 57.15 177.8) (xy 57.15 180.34)
-		)
-		(stroke
-			(width 0)
-			(type default)
-		)
-	)
 	(wire
 		(pts
@@
 		)
 	)
+	(bus
+		(pts
+			(xy 57.15 161.29) (xy 57.15 162.56)
+		)
+		(stroke
+			(width 0)
+			(type default)
+		)
+	)
 	(wire
 		(pts
@@
 		)
 	)
+	(bus
+		(pts
+			(xy 57.15 162.56) (xy 57.15 165.1)
+		)
+		(stroke
+			(width 0)
+			(type default)
+		)
+	)
 	(polyline
 		(pts
@@
 		)
 	)
+	(bus
+		(pts
+			(xy 57.15 165.1) (xy 57.15 170.18)
+		)
+		(stroke
+			(width 0)
+			(type default)
+		)
+	)
 	(wire
 		(pts
@@
 		)
 	)
+	(bus
+		(pts
+			(xy 57.15 172.72) (xy 57.15 175.26)
+		)
+		(stroke
+			(width 0)
+			(type default)
+		)
+	)
 	(wire
 		(pts
@@
 		)
 	)
+	(bus
+		(pts
+			(xy 57.15 170.18) (xy 57.15 172.72)
+		)
+		(stroke
+			(width 0)
+			(type default)
+		)
+	)
 	(wire
 		(pts
@@
 		)
 	)
-	(bus
-		(pts
-			(xy 57.15 180.34) (xy 57.15 185.42)
-		)
-		(stroke
-			(width 0)
-			(type default)
-		)
-	)
 	(wire
 		(pts
@@
 		)
 	)
+	(bus
+		(pts
+			(xy 57.15 175.26) (xy 57.15 177.8)
+		)
+		(stroke
+			(width 0)
+			(type default)
+		)
+	)
 	(wire
 		(pts
@@
 		)
 	)
-	(wire
-		(pts
-			(xy 53.34 187.96) (xy 54.61 187.96)
-		)
-		(stroke
-			(width 0)
-			(type default)
-		)
-	)
 	(bus
 		(pts
@@
 		)
 	)
-	(wire
+	(bus
 		(pts
-			(xy 72.39 175.26) (xy 73.66 175.26)
+			(xy 57.15 177.8) (xy 57.15 180.34)
 		)
 		(stroke
@@
 	(wire
 		(pts
-			(xy 167.64 175.26) (xy 172.72 175.26)
+			(xy 72.39 175.26) (xy 73.66 175.26)
 		)
 		(stroke
@@
 		)
 	)
-	(bus
+	(wire
 		(pts
-			(xy 57.15 161.29) (xy 57.15 162.56)
+			(xy 167.64 175.26) (xy 172.72 175.26)
 		)
 		(stroke
@@
 		)
 	)
+	(label "SHARED_GPIOs_SEL"
+		(at 53.34 187.96 180)
+		(effects
+			(font
+				(size 1.27 1.27)
+			)
+			(justify right bottom)
+		)
+	)
 	(label "VQPS_FUSE_1V8"
 		(at 55.88 20.32 180)
@@
 		)
 	)
-	(label "SHARED_GPIOs_SEL"
-		(at 53.34 187.96 180)
-		(effects
-			(font
-				(size 1.27 1.27)
-			)
-			(justify right bottom)
-		)
-	)
 	(label "MSP_DR2"
 		(at 175.26 72.39 0)
@@
 		(at 201.93 95.25 0)
 		(unit 1)
-		(exclude_from_sim no)
-		(in_bom yes)
-		(on_board yes)
-		(dnp no)
+		(exclude_from_sim yes)
+		(in_bom no)
+		(on_board no)
+		(dnp yes)
 		(property "Reference" "J6"
 			(at 220.726 91.186 0)
@@
 		(at 53.34 101.6 0)
 		(unit 1)
-		(exclude_from_sim no)
-		(in_bom yes)
-		(on_board yes)
-		(dnp no)
+		(exclude_from_sim yes)
+		(in_bom no)
+		(on_board no)
+		(dnp yes)
 		(property "Reference" "J5"
 			(at 72.136 97.536 0)

Commit message: V1 of pcb layout
Parts:
- removed J5: DF40C-40DP-0.4V_51, Connector_Hirose_DF40:Hirose_DF40C-40DS-0.4V_2x20_P0.4mm, symbol dz_con:DF40C-40DP-0.4V_51
- removed J6: DF40C-50DP-0.4V_51, Connector_Hirose_DF40:Hirose_DF40C-50DS-0.4V_2x25_P0.4mm, symbol dz_con:DF40C-50DP-0.4V_51
Connections:
- net ADS_A_DR: no longer names the net of J4.43
- net ADS_B_DR: no longer names the net of J4.45
- net CSI_CLK_N: no longer names the net of J3.17
- net CSI_CLK_P: no longer names the net of J3.19
- net CSI_D0_N: no longer names the net of J3.23
- net CSI_D0_P: no longer names the net of J3.25
- net EXT_CHG/VUSB: no longer names the net of J4.6
- net EXT_CHG/VUSB: no longer J4.8
- net GAP_GPIO47: no longer names the net of J3.31
- net GAP_GPIO48: no longer names the net of J3.37
- net GAP_GPIO49: no longer names the net of J3.39
- net GAP_GPIO50: no longer names the net of J3.33
- net GAP_GPIO51: no longer names the net of J3.35
- net I2C_A_SCL: no longer names the net of J4.30
- net I2C_A_SDA: no longer names the net of J4.32
- net I2C_B_SCL: no longer names the net of J4.42
- net I2C_B_SDA: no longer names the net of J4.38
- net MIC_CLK: no longer names the net of J3.36
- net MIC_DATA: no longer names the net of J3.34
- net MIC_THSEL: no longer names the net of J3.38
- net MIC_WAKE: no longer names the net of J3.40
- net MSP_CS: no longer names the net of J4.23
- net MSP_DR1: no longer names the net of J4.25
- net MSP_DR2: no longer names the net of J4.41
- net MSP_TCK: no longer names the net of J4.4
- net MSP_TDI: no longer names the net of J4.24
- net MSP_TDO: no longer names the net of J4.26
- net MSP_TMS: no longer names the net of J4.22
- net MSP_VCC: no longer names the net of J4.28
- net MSP_~{TRST}: no longer names the net of J4.2
- net QVAR_IMU_1: no longer names the net of J3.16
- net QVAR_IMU_2: no longer names the net of J3.18
- net RESET_N: no longer names the net of J3.1
- net SPI_A_CS: no longer names the net of J4.46
- net SPI_B_CLK: no longer names the net of J4.48
- net SPI_B_CS: no longer names the net of J4.47
- net SPI_B_MISO: no longer names the net of J4.50
- net SPI_B_MOSI: no longer names the net of J4.49
- net SWDCLK: no longer names the net of J4.12
- net SWDIO: no longer names the net of J4.10
- net SWO: no longer names the net of J4.14
- net TCK: no longer names the net of J3.5
- net TCS/CS_RAM_GATE: no longer names the net of J3.7
- net TDI: no longer names the net of J3.9
- net TDO: no longer names the net of J3.11
- net VA0: no longer names the net of J4.20
- net VA1: no longer names the net of J4.21
- net VBAT: no longer names the net of J4.1
- net VBAT: no longer J4.3
- net VCC_GAP9: no longer names the net of J3.13
- net VD0: no longer names the net of J4.18
- net VD1: no longer names the net of J4.17
- net VQPS_FUSE_1V8: no longer names the net of J3.14
- net VSYS: no longer names the net of J4.5
- net VSYS: no longer J4.7
- net nRF_P0.05: no longer names the net of J3.22
- net nRF_P0.07: no longer names the net of J3.26
- net nRF_P0.31: no longer names the net of J3.2
- net nRF_P1.00_GAP_GPIO60: no longer names the net of J3.4
- net nRF_P1.01_GAP_GPIO61: no longer names the net of J3.6
- net nRF_P1.09_GAP_GPIO62: no longer names the net of J3.8
- net nRF_P1.12_GAP_GPIO64 renamed nRF_P0.12_GAP_GPIO64
- net nRF_QSPI_CLK: no longer names the net of J4.39
- net nRF_QSPI_CS_CONN: no longer names the net of J4.27
- net nRF_QSPI_IO0: no longer names the net of J4.37
- net nRF_QSPI_IO1: no longer names the net of J4.33
- net nRF_QSPI_IO2: no longer names the net of J4.31
- net nRF_QSPI_IO3: no longer names the net of J4.29
- net ~{RST}: no longer names the net of J4.9
- net ~{TRST}: no longer names the net of J3.3
- no-connect marks 16 -> 73
Other:
- note removed: "40-pin board-to-board connector (female)"
- note removed: "50-pin board-to-board connector (female)"
- note removed: "Various data buses/groups"
- moved on the sheet: J3, J4

Commit message: small adjustments
Connections:
- net nRF_P0.07/AMUX: now reaches J3.26
- net 1V8 renamed 1V8_Connector
- no-connect marks 73 -> 72
Changed lines of the file:
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@@
-	)
-	(no_connect
-		(at 96.52 101.6)
 	)
 	(no_connect
@@
 		(pts
 			(xy 46.99 88.9) (xy 73.66 88.9)
+		)
+		(stroke
+			(width 0)
+			(type default)
+		)
+	)
+	(wire
+		(pts
+			(xy 96.52 101.6) (xy 107.95 101.6)
 		)
 		(stroke
@@
 		)
 	)
-	(global_label "1V8"
+	(global_label "1V8_Connector"
 		(shape output)
 		(at 162.56 76.2 180)
@@
 		)
 		(property "Intersheetrefs" "${INTERSHEET_REFS}"
-			(at 156.0672 76.2 0)
+			(at 145.5445 76.2 0)
 			(effects
 				(font
@@
 		)
 	)
-	(global_label "1V8"
+	(global_label "1V8_Connector"
 		(shape output)
 		(at 162.56 78.74 180)
@@
 		)
 		(property "Intersheetrefs" "${INTERSHEET_REFS}"
-			(at 156.0672 78.74 0)
+			(at 145.5445 78.74 0)
 			(effects
 				(font
@@
 				(hide yes)
 			)
+		)
+	)
+	(global_label "nRF_P0.07{slash}AMUX"
+		(shape bidirectional)
+		(at 107.95 101.6 0)
+		(fields_autoplaced yes)
+		(effects
+			(font
+				(size 1.27 1.27)
+			)
+			(justify left)
+		)
+		(property "Intersheetrefs" "${INTERSHEET_REFS}"
+			(at 128.4355 101.6 0)
+			(effects
+				(font
+					(size 1.27 1.27)
+				)
+				(justify left)
+				(hide yes)
+			)
