File: Hardware/mmWave-shield-pcb/mmWave-shield-pcb.kicad_pcb (KiCad board)
At the start: 4 copper layers, 21 x 15 mm, 40 parts, among them J3 DF40HC_3.0_-40DS-0.4V_51, J4 DF40HC_3.0_-50DS-0.4V_51, U1 TPS22916CYFPR, U2 TPS22916CYFPR, X1 KC2016K80.0000C1GE00

Commit message: Finish up HW cleaning
Parts:
- FB1, FB2, FB3, FB4, FB5, FB6, FB7: footprint MMZ1005S121CT000:IND_1005_TDK-L -> Project_specific_footprints:IND_1005_TDK-L
- U$1: footprint aaEXTRAS:BGA40N50P9X12_500X650X90-V -> Project_specific_footprints:BGA40N50P9X12_500X650X90-V
- U1, U2: footprint aaEXTRAS:TPS22916CYFPR -> Project_specific_footprints:TPS22916CYFPR
- X1: footprint aExtra:KC2016K_KYO -> Project_specific_footprints:KC2016K_KYO
