File: Hardware/mmWave-shield-pcb/sensor.kicad_sch (KiCad schematic)
At the start: 37 parts, among them U1 TPS22916CYFPR, U2 TPS22916CYFPR, X1 KC2016K80.0000C1GE00

Commit message: Finish up HW cleaning
Parts:
- FB1, FB2, FB3, FB4, FB5, FB6, FB7: footprint MMZ1005S121CT000:IND_1005_TDK-L -> Project_specific_footprints:IND_1005_TDK-L
- U$1: footprint aaEXTRAS:BGA40N50P9X12_500X650X90-V -> Project_specific_footprints:BGA40N50P9X12_500X650X90-V
- U1, U2: footprint aaEXTRAS:TPS22916CYFPR -> Project_specific_footprints:TPS22916CYFPR
- X1: footprint aExtra:KC2016K_KYO -> Project_specific_footprints:KC2016K_KYO
Changed lines of the file:
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@@
 			)
 		)
-		(property "Footprint" "MMZ1005S121CT000:IND_1005_TDK-L"
+		(property "Footprint" "Project_specific_footprints:IND_1005_TDK-L"
 			(at 91.44 161.798 90)
 			(effects
@@
 			)
 		)
-		(property "Footprint" "MMZ1005S121CT000:IND_1005_TDK-L"
+		(property "Footprint" "Project_specific_footprints:IND_1005_TDK-L"
 			(at 138.43 133.858 90)
 			(effects
@@
 			)
 		)
-		(property "Footprint" "MMZ1005S121CT000:IND_1005_TDK-L"
+		(property "Footprint" "Project_specific_footprints:IND_1005_TDK-L"
 			(at 247.65 39.878 90)
 			(effects
@@
 			)
 		)
-		(property "Footprint" "MMZ1005S121CT000:IND_1005_TDK-L"
+		(property "Footprint" "Project_specific_footprints:IND_1005_TDK-L"
 			(at 91.44 133.858 90)
 			(effects
@@
 			)
 		)
-		(property "Footprint" "aaEXTRAS:TPS22916CYFPR"
+		(property "Footprint" "Project_specific_footprints:TPS22916CYFPR"
 			(at 251.46 85.09 0)
 			(effects
@@
 			)
 		)
-		(property "Footprint" "aaEXTRAS:BGA40N50P9X12_500X650X90-V"
+		(property "Footprint" "Project_specific_footprints:BGA40N50P9X12_500X650X90-V"
 			(at 73.66 25.4 0)
 			(effects
@@
 			)
 		)
-		(property "Footprint" "MMZ1005S121CT000:IND_1005_TDK-L"
+		(property "Footprint" "Project_specific_footprints:IND_1005_TDK-L"
 			(at 52.07 161.798 90)
 			(effects
@@
 			)
 		)
-		(property "Footprint" "aaEXTRAS:TPS22916CYFPR"
+		(property "Footprint" "Project_specific_footprints:TPS22916CYFPR"
 			(at 187.96 86.36 0)
 			(effects
@@
 			)
 		)
-		(property "Footprint" "MMZ1005S121CT000:IND_1005_TDK-L"
+		(property "Footprint" "Project_specific_footprints:IND_1005_TDK-L"
 			(at 133.35 161.798 90)
 			(effects
@@
 			)
 		)
-		(property "Footprint" "MMZ1005S121CT000:IND_1005_TDK-L"
+		(property "Footprint" "Project_specific_footprints:IND_1005_TDK-L"
 			(at 52.07 133.858 90)
 			(effects
@@
 			)
 		)
-		(property "Footprint" "aExtra:KC2016K_KYO"
+		(property "Footprint" "Project_specific_footprints:KC2016K_KYO"
 			(at 179.07 38.1 0)
 			(effects
